File: debugger/hardware/Tek7854DBI.sch (KiCad schematic (older format))
At the start: 78 parts, among them J1 TTL SERIAL DATA, P1 SV2, P2 Tek7854_MPC_Card_Edge, P3 SV1, SW1 BUTTON 1, SW2 BUTTON 2, SW3 BUTTON 3

Commit message: NET naming error
IC1 and IC3 had incorrect net names.
Connections:
- net L47N_0 renamed L47N_1
- net L74N_0 renamed L74N_1
Changed lines of the file:
@@
 L2N_2
 Text Label 9600 2800 0    60   ~ 0
-L74N_0
+L74N_1
 Text Label 9600 2900 0    60   ~ 0
-L47N_0
+L47N_1
 Text Label 9600 3000 0    60   ~ 0
 L46N_1
